File: smd_to_dip_40/smd_to_dip_40.kicad_sch (KiCad schematic)
At the start: 2 parts, among them U1 ATmega644A-P, U2 ATmega644A-P

Commit message: commit 2
Connections:
- net PB0: now reaches U1.1 (PB0)
- net VCC: now reaches U1.10 (VCC)
- net VCC: now also U2.10 (VCC)
- net GND: now reaches U1.11 (GND), U1.31 (GND)
- net GND: now also U2.11 (GND), U2.31 (GND)
- net PB1: now reaches U1.2 (PB1)
- net PB2: now reaches U1.3 (PB2)
- net AREF: now reaches U1.32 (AREF)
- net AREF: now also U2.32 (AREF)
- net PA7: now reaches U1.33 (PA7)
- net PA6: now reaches U1.34 (PA6)
- net PA5: now reaches U1.35 (PA5)
- net PA4: now reaches U1.36 (PA4)
- net PA3: now reaches U1.37 (PA3)
- net PA2: now reaches U1.38 (PA2)
- net PA1: now reaches U1.39 (PA1)
- net PB3: now reaches U1.4 (PB3)
- net PA0: now reaches U1.40 (PA0)
- net PB4: now reaches U1.5 (PB4)
- net PB5: now reaches U1.6 (PB5)
- net PB6: now reaches U1.7 (PB6)
- net PB7: now reaches U1.8 (PB7)
Other:
- moved on the sheet: U1

Commit message: commit 3
Parts:
- added C1, C2, C3, C4: C, Capacitor_THT:C_Axial_L3.8mm_D2.6mm_P7.50mm_Horizontal, symbol Device:C
- added Y1: Crystal, Crystal:Crystal_HC18-U_Vertical, symbol Device:Crystal
Connections:
- net GND: now also C1.2, C2.2, C3.2, C4.2
- net PA0: now also U2.40 (PA0)
- net PA1: now also U2.39 (PA1)
- net PA2: now also U2.38 (PA2)
- net PA3: now also U2.37 (PA3)
- net PA4: now also U2.36 (PA4)
- net PA5: now also U2.35 (PA5)
- net PA6: now also U2.34 (PA6)
- net PA7: now also U2.33 (PA7)
- net PB0: now also U2.1 (PB0)
- net PB1: now also U2.2 (PB1)
- net PB2: now also U2.3 (PB2)
- net PB3: now also U2.4 (PB3)
- net PB4: now also U2.5 (PB4)
- net PB5: now also U2.6 (PB5)
- net PB6: now also U2.7 (PB6)
- net PB7: now also U2.8 (PB7)
- net VCC: now also C3.1, C4.1
- net XTAL1: now also C1.1, Y1.1
- net XTAL2: now also C2.1, Y1.2
- net PD0: now reaches U1.14 (PD0)
- net PD0: now also U2.14 (PD0)
- net PD1: now reaches U1.15 (PD1)
- net PD1: now also U2.15 (PD1)
- net PD2: now reaches U1.16 (PD2)
- net PD2: now also U2.16 (PD2)
- net PD3: now reaches U1.17 (PD3)
- net PD3: now also U2.17 (PD3)
- net PD4: now reaches U1.18 (PD4)
- net PD4: now also U2.18 (PD4)
- net PD5: now reaches U1.19 (PD5)
- net PD5: now also U2.19 (PD5)
- net PD6: now reaches U1.20 (PD6)
- net PD6: now also U2.20 (PD6)
- net PD7: now reaches U1.21 (PD7)
- net PD7: now also U2.21 (PD7)
- net PC0: now reaches U1.22 (PC0)
- net PC0: now also U2.22 (PC0)
- net PC1: now reaches U1.23 (PC1)
- net PC1: now also U2.23 (PC1)
- net PC2: now reaches U1.24 (PC2)
- net PC2: now also U2.24 (PC2)
- net PC3: now reaches U1.25 (PC3)
- net PC3: now also U2.25 (PC3)
- net PC4: now reaches U1.26 (PC4)
- net PC4: now also U2.26 (PC4)
- net PC5: now reaches U1.27 (PC5)
- net PC5: now also U2.27 (PC5)
- net PC6: now reaches U1.28 (PC6)
- net PC6: now also U2.28 (PC6)
- net PC7: now reaches U1.29 (PC7)
- net PC7: now also U2.29 (PC7)

Commit message: commit 4
Parts:
- added J1: Conn_02x03_Odd_Even, Connector_IDC:IDC-Header_2x03_P2.54mm_Vertical, symbol Connector_Generic:Conn_02x03_Odd_Even
Connections:
- net GND: now also J1.6 (Pin_6)
- net RESET: now also J1.5 (Pin_5)
- net VCC: now also J1.2 (Pin_2)
- net PB5 renamed PB5/MOSI
- net PB5/MOSI: now also J1.4 (Pin_4)
- net PB6 renamed PB6/MISO
- net PB6/MISO: now also J1.1 (Pin_1)
- net PB7 renamed PB7/SCK
- net PB7/SCK: now also J1.3 (Pin_3)
